File: wc/wc.kicad_pcb (KiCad board)
At the start: 2 copper layers, 98 x 98 mm, 10 parts, among them J1 USB_C_Receptacle_USB2.0, U1 XKT-510

Commit message: update: 更新
Parts:
- added ?: , , F.Cu at (134.0, 74.0)
- added ?: , , F.Cu at (44.0, 164.0)
- added ?: , , F.Cu at (44.0, 74.0)
- added ?: , , F.Cu at (134.0, 164.0)
- moved J1 1.70 mm to (44.4, 83.0)
- moved R1 1.70 mm to (49.8, 81.8)
- moved R2 1.70 mm to (49.8, 84.8)
Routing:
- net +5V: track 3427.2 -> 3426.3 mm, vias 3 -> 4
- net (no net): vias 1 -> 0

Commit message: fix: 更正参数
Parts:
- removed ? (x4): , 
- C1: value 22uf -> 22uf/16V; footprint Capacitor_SMD:C_0402_1005Metric -> Capacitor_SMD:C_0805_2012Metric
- R3: value 5.6K -> 6.2K
- moved C1 0.45 mm to (42.0, 118.8)
