File: wc/wc.kicad_sch (KiCad schematic)
At the start: 10 parts, among them J1 USB_C_Receptacle_USB2.0, U1 XKT-510

Commit message: fix: 更正参数
Parts:
- C1: value 22uf -> 22uf/16V; footprint Capacitor_SMD:C_0402_1005Metric -> Capacitor_SMD:C_0805_2012Metric
- R3: value 5.6K -> 6.2K
Changed lines of the file:
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@@
 (kicad_sch (version 20210621) (generator eeschema)
   (paper "A4")
+  (junction (at 59.055 24.13) (diameter 0) (color 0 0 0 0))
+  (junction (at 98.425 102.235) (diameter 0) (color 0 0 0 0))
+  (junction (at 98.425 112.395) (diameter 0) (color 0 0 0 0))
   (junction (at 67.31 93.98) (diameter 0) (color 0 0 0 0))
+  (junction (at 55.88 93.98) (diameter 0) (color 0 0 0 0))
+  (junction (at 71.12 31.75) (diameter 0) (color 0 0 0 0))
   (junction (at 43.815 62.23) (diameter 0) (color 0 0 0 0))
-  (junction (at 71.12 31.75) (diameter 0) (color 0 0 0 0))
-  (junction (at 98.425 102.235) (diameter 0) (color 0 0 0 0))
-  (junction (at 98.425 93.98) (diameter 0) (color 0 0 0 0))
-  (junction (at 59.055 24.13) (diameter 0) (color 0 0 0 0))
-  (junction (at 55.88 93.98) (diameter 0) (color 0 0 0 0))
-  (junction (at 98.425 104.775) (diameter 0) (color 0 0 0 0))
-  (junction (at 71.12 93.98) (diameter 0) (color 0 0 0 0))
-  (junction (at 98.425 112.395) (diameter 0) (color 0 0 0 0))
   (junction (at 62.23 93.98) (diameter 0) (color 0 0 0 0))
   (junction (at 62.23 107.315) (diameter 0) (color 0 0 0 0))
+  (junction (at 71.12 93.98) (diameter 0) (color 0 0 0 0))
+  (junction (at 98.425 93.98) (diameter 0) (color 0 0 0 0))
+  (junction (at 98.425 104.775) (diameter 0) (color 0 0 0 0))
   (no_connect (at 59.055 44.45))
+  (no_connect (at 59.055 52.07))
+  (no_connect (at 59.055 54.61))
   (no_connect (at 59.055 41.91))
   (no_connect (at 59.055 39.37))
   (no_connect (at 59.055 36.83))
-  (no_connect (at 59.055 52.07))
-  (no_connect (at 59.055 54.61))
+  (no_connect (at 71.12 104.775))
   (no_connect (at 85.09 109.855))
-  (no_connect (at 71.12 104.775))
   (wire (pts (xy 69.85 29.21) (xy 71.12 29.21))
     (stroke (width 0) (type default) (color 0 0 0 0))
@@
     (stroke (width 0) (type default) (color 0 0 0 0))
   )
+  (wire (pts (xy 71.12 31.75) (xy 71.12 33.02))
+    (stroke (width 0) (type default) (color 0 0 0 0))
+  )
   (wire (pts (xy 69.85 31.75) (xy 71.12 31.75))
     (stroke (width 0) (type default) (color 0 0 0 0))
   )
-  (wire (pts (xy 71.12 31.75) (xy 71.12 33.02))
+  (wire (pts (xy 67.31 93.98) (xy 71.12 93.98))
     (stroke (width 0) (type default) (color 0 0 0 0))
   )
@@
     (stroke (width 0) (type default) (color 0 0 0 0))
   )
-  (wire (pts (xy 67.31 93.98) (xy 71.12 93.98))
-    (stroke (width 0) (type default) (color 0 0 0 0))
-  )
   (wire (pts (xy 62.23 93.98) (xy 62.23 99.06))
     (stroke (width 0) (type default) (color 0 0 0 0))
@@
     (stroke (width 0) (type default) (color 0 0 0 0))
   )
+  (wire (pts (xy 109.22 99.695) (xy 109.22 93.98))
+    (stroke (width 0) (type default) (color 0 0 0 0))
+  )
+  (wire (pts (xy 98.425 93.98) (xy 109.22 93.98))
+    (stroke (width 0) (type default) (color 0 0 0 0))
+  )
   (wire (pts (xy 71.12 93.98) (xy 98.425 93.98))
     (stroke (width 0) (type default) (color 0 0 0 0))
   )
-  (wire (pts (xy 109.22 99.695) (xy 109.22 93.98))
-    (stroke (width 0) (type default) (color 0 0 0 0))
-  )
-  (wire (pts (xy 98.425 93.98) (xy 109.22 93.98))
-    (stroke (width 0) (type default) (color 0 0 0 0))
-  )
   (wire (pts (xy 98.425 102.235) (xy 98.425 104.775))
     (stroke (width 0) (type default) (color 0 0 0 0))
   )
+  (wire (pts (xy 45.72 99.06) (xy 45.72 93.98))
+    (stroke (width 0) (type default) (color 0 0 0 0))
+  )
   (wire (pts (xy 45.72 93.98) (xy 55.88 93.98))
-    (stroke (width 0) (type default) (color 0 0 0 0))
-  )
-  (wire (pts (xy 45.72 99.06) (xy 45.72 93.98))
     (stroke (width 0) (type default) (color 0 0 0 0))
   )
@@
   )
   (symbol (lib_id "Device:C") (at 45.72 102.87 0) (unit 1)
-    (in_bom yes) (on_board yes) (fields_autoplaced)
+    (in_bom yes) (on_board yes)
     (property "Reference" "C1" (id 0) (at 48.641 101.9615 0)
       (effects (font (size 1.27 1.27)) (justify left))
     )
-    (property "Value" "22uf" (id 1) (at 48.641 104.7366 0)
-      (effects (font (size 1.27 1.27)) (justify left))
-    )
-    (property "Footprint" "Capacitor_SMD:C_0402_1005Metric" (id 2) (at 46.6852 106.68 0)
+    (property "Value" "22uf/16V" (id 1) (at 45.72 105.41 0)
+      (effects (font (size 1.27 1.27)) (justify left))
+    )
+    (property "Footprint" "Capacitor_SMD:C_0805_2012Metric" (id 2) (at 46.6852 106.68 0)
       (effects (font (size 1.27 1.27)) hide)
     )
@@
     (in_bom yes) (on_board yes)
     (property "Reference" "R3" (id 0) (at 88.9 102.87 90))
-    (property "Value" "5.6K" (id 1) (at 90.17 104.775 90))
+    (property "Value" "6.2K" (id 1) (at 90.17 104.775 90))
     (property "Footprint" "Resistor_SMD:R_0402_1005Metric" (id 2) (at 90.17 106.553 90)
       (effects (font (size 1.27 1.27)) hide)
@@
     )
     (path "/07355698-4d9f-469b-8eac-fcd9469e9723"
-      (reference "C1") (unit 1) (value "22uf") (footprint "Capacitor_SMD:C_0402_1005Metric")
+      (reference "C1") (unit 1) (value "22uf/16V") (footprint "Capacitor_SMD:C_0805_2012Metric")
     )
     (path "/ce558228-ed2d-4fff-be71-f53d8a9d1385"
@@
     )
     (path "/261d963f-6dc2-4cec-b815-12361f934198"
-      (reference "R3") (unit 1) (value "5.6K") (footprint "Resistor_SMD:R_0402_1005Metric")
+      (reference "R3") (unit 1) (value "6.2K") (footprint "Resistor_SMD:R_0402_1005Metric")
     )
     (path "/abd02a53-118c-4362-a94e-93cc798742ab"
